File: electronics/ControlPCB/ControlPCB.kicad_pcb (KiCad board)
At the start: 2 copper layers, 119.6 x 90.4 mm, 44 parts, among them CON1 12VINPUT, P1 Opto1, P2 Opto2, P3 Opto3, P4 Opto4, P5 Opto5, P6 Opto6, P7 Tool, U1 POLOLU_A4988, U2 POLOLU_A4988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

Commit message: added attachment points to jumper ground net to isolated fill area
Parts:
- added REF**: Pin_Header_Straight_1x01, ControlPCB:Pin_Header_Straight_1x01, F.Cu at (201.9, 125.5)
- added REF**: Pin_Header_Straight_1x01, ControlPCB:Pin_Header_Straight_1x01, F.Cu at (182.9, 115.7)
Changed lines of the file:
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@@
-(kicad_pcb (version 4) (host pcbnew 4.0.2-4+6225~38~ubuntu15.10.1-stable)
+(kicad_pcb (version 4) (host pcbnew 4.0.2-stable)
   (general
-    (links 170)
+    (links 172)
     (no_connects 1)
     (area 86.030999 53.264999 208.005 149.91552)
@@
     (tracks 350)
     (zones 0)
-    (modules 44)
+    (modules 46)
     (nets 71)
   )
@@
     (mod_text_size 1 1)
     (mod_text_width 0.15)
-    (pad_size 3 3)
-    (pad_drill 3)
+    (pad_size 2.2352 2.2352)
+    (pad_drill 1.016)
     (pad_to_mask_clearance 0.2)
     (aux_axis_origin 0 0)
@@
     (add_net VCC)
   )
+  (module ControlPCB:Pin_Header_Straight_1x01 (layer F.Cu)
+    (at 201.93 125.476)
+    (descr "Through hole pin header")
+    (tags "pin header")
+    (fp_text reference REF** (at 0 -5.1) (layer F.SilkS)
+      (effects (font (size 1 1) (thickness 0.15)))
+    )
+    (fp_text value Pin_Header_Straight_1x01 (at 0 -3.1) (layer F.Fab) hide
+      (effects (font (size 1 1) (thickness 0.15)))
+    )
+    (fp_line (start 1.55 -1.55) (end 1.55 0) (layer F.Fab) (width 0.15))
+    (fp_line (start -1.75 -1.75) (end -1.75 1.75) (layer F.CrtYd) (width 0.05))
+    (fp_line (start 1.75 -1.75) (end 1.75 1.75) (layer F.CrtYd) (width 0.05))
+    (fp_line (start -1.75 -1.75) (end 1.75 -1.75) (layer F.CrtYd) (width 0.05))
+    (fp_line (start -1.75 1.75) (end 1.75 1.75) (layer F.CrtYd) (width 0.05))
+    (fp_line (start -1.55 0) (end -1.55 -1.55) (layer F.Fab) (width 0.15))
+    (fp_line (start -1.55 -1.55) (end 1.55 -1.55) (layer F.Fab) (width 0.15))
+    (fp_line (start -1.27 1.27) (end 1.27 1.27) (layer F.Fab) (width 0.15))
+    (pad 1 thru_hole circle (at 0 0) (size 2.2352 2.2352) (drill 1.016) (layers *.Cu *.Mask F.SilkS)
+      (net 1 GND))
+    (model Pin_Headers.3dshapes/Pin_Header_Straight_1x01.wrl
+      (at (xyz 0 0 0))
+      (scale (xyz 1 1 1))
+      (rotate (xyz 0 0 90))
+    )
+  )
   (module Symbols:Symbol_OSHW-Logo_CopperTop_BIG (layer F.Cu)
     (at 109.22 116.84)
@@
     (pad 1 thru_hole circle (at 0 0) (size 3 3) (drill 3) (layers *.Cu *.Mask F.SilkS))
   )
+  (module ControlPCB:Pin_Header_Straight_1x01 (layer F.Cu)
+    (at 182.88 115.697)
+    (descr "Through hole pin header")
+    (tags "pin header")
+    (fp_text reference REF** (at 0 -5.1) (layer F.SilkS)
+      (effects (font (size 1 1) (thickness 0.15)))
+    )
+    (fp_text value Pin_Header_Straight_1x01 (at 0 -3.1) (layer F.Fab) hide
+      (effects (font (size 1 1) (thickness 0.15)))
+    )
+    (fp_line (start 1.55 -1.55) (end 1.55 0) (layer F.Fab) (width 0.15))
+    (fp_line (start -1.75 -1.75) (end -1.75 1.75) (layer F.CrtYd) (width 0.05))
+    (fp_line (start 1.75 -1.75) (end 1.75 1.75) (layer F.CrtYd) (width 0.05))
+    (fp_line (start -1.75 -1.75) (end 1.75 -1.75) (layer F.CrtYd) (width 0.05))
+    (fp_line (start -1.75 1.75) (end 1.75 1.75) (layer F.CrtYd) (width 0.05))
+    (fp_line (start -1.55 0) (end -1.55 -1.55) (layer F.Fab) (width 0.15))
+    (fp_line (start -1.55 -1.55) (end 1.55 -1.55) (layer F.Fab) (width 0.15))
+    (fp_line (start -1.27 1.27) (end 1.27 1.27) (layer F.Fab) (width 0.15))
+    (pad 1 thru_hole circle (at 0 0) (size 2.2352 2.2352) (drill 1.016) (layers *.Cu *.Mask F.SilkS)
+      (net 1 GND))
+    (model Pin_Headers.3dshapes/Pin_Header_Straight_1x01.wrl
+      (at (xyz 0 0 0))
+      (scale (xyz 1 1 1))
+      (rotate (xyz 0 0 90))
+    )
+  )
   (gr_line (start 199.365192 127.873248) (end 199.365192 127.873248) (layer Dwgs.User) (width 0.1))
